Commit message: 更新配置

File: src/simu/urdf/xju_model.urdf.xacro (robot description, xacro)
@@ -368,71 +368,76 @@
   </joint>
   <!-- Ultrasonic -->
-    <link name="ultra_left_front_link">
-      <visual>
-        <origin
-          xyz="0 0 0"
-          rpy="0 0 0" />
-        <geometry>
-          <box size="0.01 0.01 0.01" />
-        </geometry>
-        <material name="red" />
-      </visual>
-    </link>
-    <joint name="ultra_left_front_joint" type="fixed">
-      <axis xyz="0 0 0" />
-      <origin xyz="0.3 0.195 0.1" rpy="0 0 0.7854"/>
-      <parent link="base_link"/>
-      <child link="ultra_left_front_link"/>
-    </joint>
-    <link name="ultra_left_back_link">
-      <visual>
-        <origin
-          xyz="0 0 0"
-          rpy="0 0 0" />
-        <geometry>
-          <box size="0.01 0.01 0.01" />
-        </geometry>
-        <material name="red" />
-      </visual>
-    </link>
-    <joint name="ultra_left_back_joint" type="fixed">
-      <axis xyz="0 0 0" />
-      <origin xyz="-0.1 0.195 0.1" rpy="0 0 2.3562"/>
-      <parent link="base_link"/>
-      <child link="ultra_left_back_link"/>
-    </joint>
-    <link name="ultra_right_back_link">
-      <visual>
-        <origin
-          xyz="0 0 0"
-          rpy="0 0 0" />
-        <geometry>
-          <box size="0.01 0.01 0.01" />
-        </geometry>
-        <material name="red" />
-      </visual>
-    </link>
-    <joint name="ultra_right_back_joint" type="fixed">
-      <axis xyz="0 0 0" />
-      <origin xyz="-0.1 -0.195 0.1" rpy="0 0 -2.3562"/>
-      <parent link="base_link"/>
-      <child link="ultra_right_back_link"/>
-    </joint>
-    <link name="ultra_right_front_link">
-      <visual>
-        <origin
-          xyz="0 0 0"
-          rpy="0 0 0" />
-        <geometry>
-          <box size="0.01 0.01 0.01" />
-        </geometry>
-        <material name="red" />
-      </visual>
-    </link>
-    <joint name="ultra_right_front_joint" type="fixed">
-      <axis xyz="0 0 0" />
-      <origin xyz="0.3 -0.195 0.1" rpy="0 0 -0.7854"/>
-      <parent link="base_link"/>
-      <child link="ultra_right_front_link"/>
-    </joint>
+  <link name="ultra_left_front_link">
+    <visual>
+      <origin
+        xyz="0 0 0"
+        rpy="0 0 0" />
+      <geometry>
+        <box size="0.01 0.01 0.01" />
+      </geometry>
+      <material name="red" />
+    </visual>
+  </link>
+  <joint name="ultra_left_front_joint" type="fixed">
+    <axis xyz="0 0 0" />
+    <origin xyz="0.3 0.195 0.1" rpy="0 0 0.7854"/>
+    <parent link="base_link"/>
+    <child link="ultra_left_front_link"/>
+  </joint>
+  <link name="ultra_left_back_link">
+    <visual>
+      <origin
+        xyz="0 0 0"
+        rpy="0 0 0" />
+      <geometry>
+        <box size="0.01 0.01 0.01" />
+      </geometry>
+      <material name="red" />
+    </visual>
+  </link>
+  <joint name="ultra_left_back_joint" type="fixed">
+    <axis xyz="0 0 0" />
+    <origin xyz="-0.1 0.195 0.1" rpy="0 0 2.3562"/>
+    <parent link="base_link"/>
+    <child link="ultra_left_back_link"/>
+  </joint>
+  <link name="ultra_right_back_link">
+    <visual>
+      <origin
+        xyz="0 0 0"
+        rpy="0 0 0" />
+      <geometry>
+        <box size="0.01 0.01 0.01" />
+      </geometry>
+      <material name="red" />
+    </visual>
+  </link>
+  <joint name="ultra_right_back_joint" type="fixed">
+    <axis xyz="0 0 0" />
+    <origin xyz="-0.1 -0.195 0.1" rpy="0 0 -2.3562"/>
+    <parent link="base_link"/>
+    <child link="ultra_right_back_link"/>
+  </joint>
+  <link name="ultra_right_front_link">
+    <visual>
+      <origin
+        xyz="0 0 0"
+        rpy="0 0 0" />
+      <geometry>
+        <box size="0.01 0.01 0.01" />
+      </geometry>
+      <material name="red" />
+    </visual>
+  </link>
+  <joint name="ultra_right_front_joint" type="fixed">
+    <axis xyz="0 0 0" />
+    <origin xyz="0.3 -0.195 0.1" rpy="0 0 -0.7854"/>
+    <parent link="base_link"/>
+    <child link="ultra_right_front_link"/>
+  </joint>
+  <link name="dummy"/>
+  <joint name="dummy_joint" type="fixed">
+    <parent link="dummy"/>
+    <child link="base_link"/>
+  </joint>
 </robot>
